Commit message: la table avec le rail qui bouge est faite

File: src/franka_11_description/urdf/fr3_on_table.xacro (robot description, xacro)
@@ -1,49 +1,51 @@
 <?xml version="1.0"?>
-<robot xmlns:xacro="http://ros.org/wiki/xacro" name="fr3_on_table">
-  <!-- ===================== -->
-  <!-- Include Franka macros -->
-  <!-- ===================== -->
-  <xacro:include
-    filename="$(find franka_description)/robots/common/franka_robot.xacro"/>
-  <!-- ===================== -->
+<robot xmlns:xacro="http://ros.org/wiki/xacro" name="table_rail_montage">
   <!-- Table -->
-  <!-- ===================== -->
   <link name="table">
     <visual>
       <origin xyz="0 0 0.5"/>
-      <geometry>
-        <box size="1 1 1"/>
-      </geometry>
-      <material name="grey">
-        <color rgba="0.6 0.6 0.6 1.0"/>
-      </material>
+      <geometry><box size="0.5 2 1"/></geometry>
+      <material name="grey"><color rgba="0.6 0.6 0.6 1.0"/></material>
     </visual>
     <collision>
       <origin xyz="0 0 0.5"/>
-      <geometry>
-        <box size="1 1 1"/>
-      </geometry>
+      <geometry><box size="0.5 2 1"/></geometry>
     </collision>
-    <inertial>
-      <origin xyz="0 0 0.5"/>
-      <mass value="100"/>
-      <inertia
-        ixx="10" ixy="0" ixz="0"
-        iyy="10" iyz="0"
-        izz="10"/>
-    </inertial>
   </link>
-  <!-- ===================== -->
-  <!-- Instantiate FR3 -->
-  <!-- ===================== -->
-  <xacro:franka_robot
-    arm_id="fr3"
-    parent="table"
-    joint_limits="${xacro.load_yaml('$(find franka_description)/robots/fr3/joint_limits.yaml')}"
-    inertials="${xacro.load_yaml('$(find franka_description)/robots/fr3/inertials.yaml')}"
-    kinematics="${xacro.load_yaml('$(find franka_description)/robots/fr3/kinematics.yaml')}"
-    accelerometer_config="${xacro.load_yaml('$(find franka_description)/robots/fr3/accelerometers.yaml')}"
-    dynamics="${xacro.load_yaml('$(find franka_description)/robots/fr3/dynamics.yaml')}"
-    xyz="0 0 1.0"
-    rpy="0 0 0"/>
+  <!-- Rail sur la table-->
+  <link name="rail">
+    <visual>
+      <origin xyz="0 0 1.01"/>
+      <geometry><box size="0.20 1.9 0.02"/></geometry>
+      <material name="blue"><color rgba="0 0 1 1.0"/></material>
+    </visual>
+    <collision>
+      <origin xyz="0 0 1.01"/>
+      <geometry><box size="0.20 1.9 0.02"/></geometry>
+    </collision>
+  </link>
+  <joint name="table_to_rail" type="fixed">
+    <parent link="table"/>
+    <child link="rail"/>
+    <origin xyz="0 0 0"/>
+  </joint>
+  <!-- La pièce qui glisse ("montage") -->
+  <link name="montage">
+    <visual>
+      <origin xyz="0.0 0 1.03"/>
+      <geometry><box size="0.2 0.2 0.02"/></geometry>
+      <material name="red"><color rgba="1 0 0 1.0"/></material>
+    </visual>
+    <collision>
+      <origin xyz="0.0 0 1.03"/>
+      <geometry><box size="0.2 0.2 0.02"/></geometry>
+    </collision>
+  </link>
+  <joint name="rail_joint" type="prismatic">
+    <origin xyz="0 -0.95 0" rpy="0 0 0"/>
+    <parent link="rail"/>
+    <child link="montage"/>
+    <axis xyz="0 1 0"/>
+    <limit lower="0" upper="1.9" effort="1000" velocity="0.5"/>
+  </joint>
 </robot>

File: src/franka_11_description/urdf/rail.xacro (robot description, xacro)
@@ -5,8 +5,8 @@
       <visual>
         <geometry>
-          <box size="1.5 0.2 0.1"/>
+          <box size="0.25 2 0.1"/>
         </geometry>
-        <material name="Cyan">
-            <color rgba="0 1.0 1.0 1.0"/>
+        <material name="blue">
+            <color rgba="0 0 1.0 1.0"/>
         </material>
       </visual>

File: src/franka_11_description/urdf/table.xacro (robot description, xacro)
@@ -14,5 +14,5 @@
     </link>
     <joint name="table_fixed" type="fixed">
-      <parent link="${parent}"/>
+      <parent link="base"/>
       <child link="table"/>
     </joint>
