Commit message: premier essai de rajouter le robot = failure

File: src/franka_11_description/urdf/fr3_sur_rail.urdf.xacro (robot description, xacro)
@@ -1,14 +1,12 @@
 <?xml version="1.0"?>
-<robot xmlns:xacro="http://www.ros.org/wiki/xacro" name="fr3_on_rail">
+<robot xmlns:xacro="http://www.ros.org/wiki/xacro" name="fr3_sur_rail">
   <xacro:include filename="$(find franka_description)/robots/fr3/fr3.urdf.xacro"/>
-  <xacro:include filename="$(find franka_11_description)/urdf/rail.xacro"/>
-  <xacro:include filename="$(find franka_11_description)/urdf/table.xacro"/>
-  <link name="world"/>
-  <!-- Environment -->
-  <xacro:table parent="world"/>
-  <xacro:rail parent="table"/>
+  <xacro:include filename="$(find franka_11_description)/urdf/rail_sur_table.xacro"/>
   <!-- Robot -->
-  <xacro:franka_robot
+    <xacro:franka_robot
     arm_id="fr3"
+    parent="montage"
+    xyz="0 0 0"
+    rpy="0 0 0"
     joint_limits="${xacro.load_yaml('$(find franka_description)/robots/fr3/joint_limits.yaml')}"
     inertials="${xacro.load_yaml('$(find franka_description)/robots/fr3/inertials.yaml')}"
@@ -16,6 +14,4 @@
     accelerometer_config="${xacro.load_yaml('$(find franka_description)/robots/fr3/accelerometers.yaml')}"
     dynamics="${xacro.load_yaml('$(find franka_description)/robots/fr3/dynamics.yaml')}"
-    connected_to="rail_carriage"
-    use_fake_hardware="true"
   />
 </robot>
