Commit message: Simulation avec JointStatePublisher GUI

File: src/franka_11_description/urdf/fr3_sur_rail.xacro (robot description, xacro)
@@ -1,10 +1,14 @@
 <?xml version="1.0"?>
-<robot xmlns:xacro="http://www.ros.org/wiki/xacro" name="fr3_sur_rail">
-  <xacro:include filename="$(find franka_description)/robots/fr3/fr3.urdf.xacro"/>
+<robot xmlns:xacro="http://ros.org/wiki/xacro" name="fr3_sur_rail">
+  <!-- ===================== -->
+  <!-- Includes -->
+  <!-- ===================== -->
+  <xacro:include filename="$(find franka_description)/robots/common/franka_robot.xacro"/>
   <xacro:include filename="$(find franka_11_description)/urdf/rail_sur_table.xacro"/>
+  <!-- ===================== -->
   <!-- Robot -->
-    <xacro:franka_robot
+  <!-- ===================== -->
+  <xacro:franka_robot
     arm_id="fr3"
-    parent="montage"
     xyz="0 0 0"
     rpy="0 0 0"
@@ -15,3 +19,12 @@
     dynamics="${xacro.load_yaml('$(find franka_description)/robots/fr3/dynamics.yaml')}"
   />
+  <!-- ===================== -->
+  <!-- Attacher le robot au montage -->
+  <!-- ===================== -->
+  <joint name="montage_to_base" type="fixed">
+    <origin xyz="0 0 1.04" rpy="0 0 0"/>
+    <parent link="montage"/>
+    <child link="base"/>
+    <origin xyz="0 0 0" rpy="0 0 0"/>
+  </joint>
 </robot>
